Commit message: Update README and enhance Gazebo configuration for Thundercar simulation
- Expanded README to clarify the use of Gazebo ground-truth odometry and added instructions for checking odometry and TF configurations.
- Updated package.xml to include std_msgs as a dependency.
- Improved ackermann_to_twist.py to ensure correct steering angle preservation and prevent stale command issues.
- Enhanced odom_to_tf.py to enforce canonical frame names for odometry transformations.
- Modified tc.gazebo.xacro to improve Ackermann steering plugin configuration and added a ground-truth odometry publisher.
- Adjusted wheel and chassis URDF configurations for better simulation performance and collision handling.
- Updated ros_gz_bridge configuration to include wheel-integrated odometry for diagnostics.

File: src/tc_description/urdf/tc.gazebo.xacro (robot description, xacro)
@@ -3,14 +3,19 @@
   <!-- Gazebo Harmonic plugins and RGB-D sensors for Thundercar -->
   <xacro:macro name="thundercar_gazebo">
-    <!-- Chassis friction / contact -->
+    <!-- Chassis: keep collision off the ground so it does not scrape/slide -->
     <gazebo reference="base_link">
-      <mu1>0.2</mu1>
-      <mu2>0.2</mu2>
+      <mu1>0.0</mu1>
+      <mu2>0.0</mu2>
     </gazebo>
-    <!-- Ackermann steering (rear drive, front steer) -->
+    <!-- Single AckermannSteering: sets steer angles AND matching L/R wheel
+         speeds together (kinematically consistent — no DiffDrive scrubbing).
+         Drive all four wheels like the Gazebo ackermann_steering demo.
+         Wheel odom is demoted; ground-truth /odom comes from OdometryPublisher. -->
     <gazebo>
       <plugin filename="gz-sim-ackermann-steering-system"
               name="gz::sim::systems::AckermannSteering">
+        <left_joint>front_left_wheel_joint</left_joint>
         <left_joint>back_left_wheel_joint</left_joint>
+        <right_joint>front_right_wheel_joint</right_joint>
         <right_joint>back_right_wheel_joint</right_joint>
         <left_steering_joint>left_hinge_joint</left_steering_joint>
@@ -20,11 +25,21 @@
         <wheel_base>0.340</wheel_base>
         <wheel_radius>0.05525</wheel_radius>
-        <!-- Moderate gains: huge P can chatter steering and induce yaw drift -->
-        <steer_p_gain>100.0</steer_p_gain>
-        <steer_d_gain>10.0</steer_d_gain>
+        <steering_limit>0.6</steering_limit>
+        <steer_p_gain>10000</steer_p_gain>
         <topic>/model/thundercar/cmd_vel</topic>
-        <odom_topic>/model/thundercar/odometry</odom_topic>
+        <odom_topic>/model/thundercar/odometry_wheel</odom_topic>
         <frame_id>odom</frame_id>
         <child_frame_id>base_link</child_frame_id>
+        <odom_publish_frequency>50</odom_publish_frequency>
+        <tf_topic>/model/thundercar/tf_ackermann</tf_topic>
+      </plugin>
+    </gazebo>
+    <!-- Ground-truth odom from model world pose (canonical /odom source) -->
+    <gazebo>
+      <plugin filename="gz-sim-odometry-publisher-system"
+              name="gz::sim::systems::OdometryPublisher">
+        <odom_frame>odom</odom_frame>
+        <robot_base_frame>base_link</robot_base_frame>
+        <odom_topic>/model/thundercar/odometry</odom_topic>
         <odom_publish_frequency>50</odom_publish_frequency>
       </plugin>

File: src/tc_description/urdf/tc.urdf.xacro (robot description, xacro)
@@ -38,7 +38,7 @@
     </visual>
     <collision>
-      <origin xyz="0 0 0.02" rpy="0 0 0"/>
-      <geometry>
-        <box size="${length_body} ${width_body} ${height_body}"/>
+      <origin xyz="0 0 0.04" rpy="0 0 0"/>
+      <geometry>
+        <box size="${length_body} ${width_body} 0.04"/>
       </geometry>
     </collision>

File: src/tc_description/urdf/wheel.urdf.xacro (robot description, xacro)
@@ -51,6 +51,7 @@
     </joint>
     <gazebo reference="${rf}_${lr}_wheel">
-      <mu1>1.2</mu1>
-      <mu2>1.2</mu2>
+      <!-- Higher lateral grip so steered wheels pull the chassis into a yaw -->
+      <mu1>2.5</mu1>
+      <mu2>2.5</mu2>
       <kp>1000000.0</kp>
       <kd>100.0</kd>
@@ -86,7 +87,6 @@
       <origin xyz="${translateX * base_x_origin_to_hinge_origin} ${translateY * base_y_origin_to_hinge_origin} ${translateZ * base_z_origin_to_hinge_origin}" rpy="0 0 0"/>
       <axis xyz="0 0 1"/>
-      <limit lower="-0.6" upper="0.6" effort="50" velocity="5"/>
-      <!-- Higher damping so idle steering settles at center (reduces yaw drift) -->
-      <dynamics damping="5.0" friction="1.0"/>
+      <limit lower="-0.6" upper="0.6" effort="20" velocity="5"/>
+      <dynamics damping="0.5" friction="0.0"/>
     </joint>
   </xacro:macro>
@@ -121,6 +121,6 @@
     </joint>
     <gazebo reference="${rf}_${lr}_wheel">
-      <mu1>1.2</mu1>
-      <mu2>1.2</mu2>
+      <mu1>2.5</mu1>
+      <mu2>2.5</mu2>
       <kp>1000000.0</kp>
       <kd>100.0</kd>

Commit message: Enhance teleoperation and simulation configurations for Thundercar
- Updated teleop.launch.py to include a process for killing orphaned keyboard terminals before starting a new teleoperation session, preventing unintended vehicle movement.
- Modified keyboard_ackermann.py to adjust speed parameters and implement an idle stop feature, improving control responsiveness.
- Enhanced URDF configurations for wheels and chassis to improve simulation dynamics, including adjustments to friction and damping values.
- Updated SLAM parameters in slam_params.yaml for better lidar range matching and improved scan matching behavior.
- Added friction properties to indoor and level 16 SDF worlds to enhance vehicle interaction with surfaces.
- Improved RViz configuration for better visualization of simulation data, including adjustments to display settings and added landmarks for SLAM.

File: src/tc_description/urdf/tc.gazebo.xacro (robot description, xacro)
@@ -27,4 +27,9 @@
         <steering_limit>0.6</steering_limit>
         <steer_p_gain>10000</steer_p_gain>
+        <!-- Soft brake when cmd stops; still allows normal accel -->
+        <min_velocity>-2.0</min_velocity>
+        <max_velocity>2.0</max_velocity>
+        <min_acceleration>-4.0</min_acceleration>
+        <max_acceleration>3.0</max_acceleration>
         <topic>/model/thundercar/cmd_vel</topic>
         <odom_topic>/model/thundercar/odometry_wheel</odom_topic>

File: src/tc_description/urdf/wheel.urdf.xacro (robot description, xacro)
@@ -48,10 +48,10 @@
       <origin xyz="${translateX * base_x_origin_to_wheel_origin} ${translateY * base_y_origin_to_wheel_origin} ${translateZ * base_z_origin_to_wheel_origin}" rpy="0 0 0"/>
       <axis xyz="0 1 0"/>
-      <dynamics damping="0.1" friction="0.0"/>
+      <dynamics damping="0.5" friction="0.05"/>
     </joint>
     <gazebo reference="${rf}_${lr}_wheel">
-      <!-- Higher lateral grip so steered wheels pull the chassis into a yaw -->
-      <mu1>2.5</mu1>
-      <mu2>2.5</mu2>
+      <!-- Enough grip to resist sideways slide at rest, still driveable -->
+      <mu1>12.0</mu1>
+      <mu2>8.0</mu2>
       <kp>1000000.0</kp>
       <kd>100.0</kd>
@@ -88,5 +88,5 @@
       <axis xyz="0 0 1"/>
       <limit lower="-0.6" upper="0.6" effort="20" velocity="5"/>
-      <dynamics damping="0.5" friction="0.0"/>
+      <dynamics damping="1.0" friction="0.1"/>
     </joint>
   </xacro:macro>
@@ -118,9 +118,9 @@
       <origin xyz="0 ${translateY * 0.0165} 0" rpy="0 0 0"/>
       <axis xyz="0 1 0"/>
-      <dynamics damping="0.1" friction="0.0"/>
+      <dynamics damping="0.5" friction="0.05"/>
     </joint>
     <gazebo reference="${rf}_${lr}_wheel">
-      <mu1>2.5</mu1>
-      <mu2>2.5</mu2>
+      <mu1>12.0</mu1>
+      <mu2>8.0</mu2>
       <kp>1000000.0</kp>
       <kd>100.0</kd>
